Commit message: working on thruster plugin xacro.

File: gazebo/models/urdf/srpl_mass_on_rails_model.urdf (robot description, URDF)
Before this commit: robot srpl_mass_on_rails, 2 links, 1 joints
Links:
- added link rail1; collision box size=0.05 0.05 2.2; visual box size=0.05 0.05 2.2
- added link rail2; collision box size=0.05 0.05 2.2; visual box size=0.05 0.05 2.2
- link base: mass None -> 100; geometry collision cylinder length=0.01 radius=0.8; visual cylinder length=0.01 radius=0.8
- link mass: mass None -> 10; geometry collision box size=0.2 0.2 0.2; visual box size=0.2 0.2 0.2
Joints:
- removed joint joint
- added joint mass_base_joint: type prismatic, parent base, child mass, axis 0 0 1, limit lower=0 upper=2 effort=50 velocity=100
- added joint rail1_base_joint: type fixed, parent base, child rail1
- added joint rail2_base_joint: type fixed, parent base, child rail2
